File: RioPicoBridge/_autosave-RioPicoBridge.kicad_sch (KiCad schematic)
At the start: 19 parts, among them J1 DUPONT, J2 DUPONT, J3 JST, J5 MXP, U1 Pico, U2 LM1117-3.3

Commit message: v2
Parts:
- gave numbers to parts that had none: 1
Changed lines of the file:
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@@
   (symbol (lib_id "Connector:Conn_01x05_Female") (at 227.33 104.14 180) (unit 1)
     (in_bom yes) (on_board yes)
-    (property "Reference" "J?" (id 0) (at 227.33 93.98 0))
+    (property "Reference" "J4" (id 0) (at 227.33 93.98 0))
     (property "Value" "JST" (id 1) (at 227.33 96.52 0))
     (property "Footprint" "Connector_JST:JST_PH_S4B-PH-SM4-TB_1x04-1MP_P2.00mm_Horizontal" (id 2) (at 227.33 104.14 0)
@@
   (symbol (lib_id "power:GND") (at 240.03 101.6 90) (unit 1)
     (in_bom yes) (on_board yes) (fields_autoplaced)
-    (property "Reference" "#PWR?" (id 0) (at 246.38 101.6 0)
+    (property "Reference" "#PWR0103" (id 0) (at 246.38 101.6 0)
       (effects (font (size 1.27 1.27)) hide)
     )
@@
   (symbol (lib_id "power:+3V3") (at 240.03 104.14 270) (unit 1)
     (in_bom yes) (on_board yes) (fields_autoplaced)
-    (property "Reference" "#PWR?" (id 0) (at 236.22 104.14 0)
+    (property "Reference" "#PWR0104" (id 0) (at 236.22 104.14 0)
       (effects (font (size 1.27 1.27)) hide)
     )
@@
       (reference "#PWR0102") (unit 1) (value "GND") (footprint "")
     )
+    (path "/3203ce50-ef83-431b-a38b-f8ca07c919c5"
+      (reference "#PWR0103") (unit 1) (value "GND") (footprint "")
+    )
+    (path "/dce7196c-bf07-4052-a9de-915925ff82f4"
+      (reference "#PWR0104") (unit 1) (value "+3V3") (footprint "")
+    )
     (path "/e8e807a4-269f-4fd7-8f2b-f1b407adfd9e"
       (reference "#PWR0107") (unit 1) (value "+3V3") (footprint "")
@@
       (reference "#PWR0131") (unit 1) (value "+3V3") (footprint "")
     )
-    (path "/3203ce50-ef83-431b-a38b-f8ca07c919c5"
-      (reference "#PWR?") (unit 1) (value "GND") (footprint "")
-    )
-    (path "/dce7196c-bf07-4052-a9de-915925ff82f4"
-      (reference "#PWR?") (unit 1) (value "+3V3") (footprint "")
-    )
     (path "/16a3a2dc-f6c2-4c1d-a75e-be06c82f10ee"
       (reference "C1") (unit 1) (value "10uF") (footprint "Capacitor_SMD:C_0805_2012Metric")
@@
       (reference "J3") (unit 1) (value "JST") (footprint "Connector_JST:JST_PH_S4B-PH-SM4-TB_1x04-1MP_P2.00mm_Horizontal")
     )
+    (path "/1be135a4-7f20-4573-9c11-2e6713feb7f4"
+      (reference "J4") (unit 1) (value "JST") (footprint "Connector_JST:JST_PH_S4B-PH-SM4-TB_1x04-1MP_P2.00mm_Horizontal")
+    )
     (path "/c6339fa9-1ff0-48c4-9fce-d565bb93661c"
       (reference "J5") (unit 1) (value "MXP") (footprint "Connector_PinSocket_2.54mm:PinSocket_2x17_P2.54mm_Vertical")
     )
-    (path "/1be135a4-7f20-4573-9c11-2e6713feb7f4"
-      (reference "J?") (unit 1) (value "JST") (footprint "Connector_JST:JST_PH_S4B-PH-SM4-TB_1x04-1MP_P2.00mm_Horizontal")
-    )
     (path "/11ed9d27-5ddc-4a7d-b52c-68c3cefa5f56"
