File: RioPicoBridge/RioPicoBridge.kicad_pcb (KiCad board)
At the start: 2 copper layers, 56.7 x 77.5 mm, 13 parts, among them J1 DUPONT, J2 DUPONT, J3 JST PH, J4 JST PH, J5 MXP, U1 Pico

Commit message: v2
Parts:
- added C1: 10uF, Capacitor_SMD:C_0805_2012Metric, F.Cu at (5.45, 67.1)
- added C2: 10uF, Capacitor_SMD:C_0805_2012Metric, F.Cu at (10.0, 31.9)
- added C3: 100uF, Capacitor_SMD:C_0805_2012Metric, F.Cu at (5.47, 32.0)
- added JP1: Jumper_2_Open, Jumper:SolderJumper-2_P1.3mm_Open_TrianglePad1.0x1.5mm, F.Cu at (9.82, 35.0)
- added JP2: Jumper_2_Open, Jumper:SolderJumper-2_P1.3mm_Open_TrianglePad1.0x1.5mm, F.Cu at (6.47, 34.9)
- added U2: LM1117-3.3, Package_TO_SOT_SMD:TO-263-3_TabPin2, F.Cu at (6.65, 22.4)
- J3, J4: value JST PH -> JST
- moved J3 1.00 mm to (36.0, 15.0)
- moved J4 1.00 mm to (21.0, 15.0)
- turned R1 to 180 degrees
- turned R2 to 180 degrees
- turned R3 to 180 degrees
- turned R4 to 180 degrees
Connections:
- J3 pad MP: (no net) -> GND
- J4 pad MP: (no net) -> GND
- R1 pad 1: +3V3 -> /SCL2
- R1 pad 2: /SCL2 -> +3V3
- R2 pad 1: +3V3 -> /SDA2
- R2 pad 2: /SDA2 -> +3V3
- R3 pad 1: +3V3 -> /SDA1
- R3 pad 2: /SDA1 -> +3V3
- R4 pad 1: +3V3 -> /SCL1
- R4 pad 2: /SCL1 -> +3V3
Routing:
- net +5V: track 3.26 -> 107.4 mm, vias 0 -> 1
- net Net-(C3-Pad1): track 0.00 -> 15.2 mm
- net +3V3: track 115.8 -> 126.0 mm
- net Net-(C2-Pad1): track 0.00 -> 8.87 mm
- net /SCL2: track 39.9 -> 32.1 mm, vias 1 -> 0
- net /SCL1: track 48.0 -> 51.5 mm
- net /SCLK: track 37.7 -> 35.3 mm
- net /SDA2: track 51.2 -> 49.8 mm
- net /RIO_RX: track 47.7 -> 46.9 mm
- net GND: vias 205 -> 153
Other:
- board text added: "JUMP FOR 3V3 LDO"
- board text added: "RAHEEL R. DECEMBER 2022 V2 FOR ROBORIO MXP"
- board text added: "{ "ViaStitching": "0.1", "stitch_zone_0": { "HSpacing": "3", "VSpacing": "3", "Clearance": "1", "Randomize": false } }"
- board text removed: "RAHEEL R. OCTOBER 2022 FOR ROBORIO MXP"
- board text removed: "{ "ViaStitching": "0.1", "stitch_zone_1": { "HSpacing": "2", "VSpacing": "2", "Clearance": "2", "Randomize": false } }"

Commit message: forgot to add gerbers
Parts:
- moved C3 132.5 mm to (124.6, 90.1)
- moved J2 132.5 mm to (144.2, 82.1)
- moved JP1 132.5 mm to (128.9, 93.1)
- moved R1 132.5 mm to (138.6, 90.1)
- moved C2 132.5 mm to (129.1, 90.1)
- moved H1 132.5 mm to (172.2, 61.6)
- moved H2 132.5 mm to (122.6, 61.6)
- moved J1 132.5 mm to (159.6, 82.1)
- moved J3 132.5 mm to (155.1, 73.1)
- moved J4 132.5 mm to (140.1, 73.1)
- moved J5 132.5 mm to (167.7, 129.7)
- moved JP2 132.5 mm to (125.6, 93.0)
- moved R2 132.5 mm to (138.7, 87.6)
- moved R3 132.5 mm to (154.1, 87.1)
- moved R4 132.5 mm to (154.1, 89.6)
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Routing:
- net /SCL2: track 32.1 -> 31.2 mm
Other:
- board size 56.7 x 77.5 mm -> 56.6 x 77.5 mm
